File: EDM_Powersupply.kicad_sch (KiCad schematic)
At the start: 27 parts, among them IC1 ACSL-7210-06RE, J1 Screw_Terminal_01x02, Q1 IPW65R037C6, U1 L7805, U2 STGAP2SM, U3 RP2040, U4 MGJ2D051505SC, U6 LMV7239

Commit message: switched some things around, mainly gnds
Parts:
- removed U3: RP2040, Package_DFN_QFN:QFN-56-1EP_7x7mm_P0.4mm_EP3.2x3.2mm, symbol MCU_RaspberryPi:RP2040
- removed U6: LMV7239, Package_TO_SOT_SMD:SOT-353_SC-70-5, symbol Comparator:LMV7219M7
- added C8: 100n, symbol Device:C
- added C9: 2.2u, symbol Device:C
- added R10: 6.2k, symbol Device:R
- added R9: 22k, symbol Device:R
- added U3: RASPBERRY_PI_PICO, RASPBERRY_PI_PICO:RASPBERRY_PI_PICO, symbol RASPBERRY_PI_PICO:RASPBERRY_PI_PICO
- added U5: TLV3501AID, Package_SO:SOIC-8_3.9x4.9mm_P1.27mm, symbol Comparator:TLV3501AID
Connections:
- net +15V: now also C9.2, R9.1
- net +3.3V: now also U3.3V3
- net +5V: now also U3.VSYS
- net DigitalMeasureHigh: now also U5.6
- net DigitalMeasureLow: now also U3.GP3
- net GND: no longer C5.2, C7.2, IC1.5 (GND_2), R12.2, U4.6 (0V)
- net GNDS: now also U3.AGND, U3.GND, U3.GND2, U3.GND3, U3.GND4, U3.GND5, U3.GND6, U3.GND7
- net MeasRefPWMLow: now also U3.GP2
- net PWM: now also U3.GP0
- net at R6.2, R7.2: now also U5.3 (+)
- net at C5.1, R8.1: now also U5.2 (-)
- net GND1: now reaches Q1.3 (SOURCE), R3.1, U2.8 (GNDISO)
- net GND1: now also C5.2, C7.2, IC1.5 (GND_2), R12.2, U4.6 (0V), C8.2, C9.1, R10.2, U5.4 (V-), U5.8 (SHDN)
- new net: C8.1, R10.1, R9.2, U5.7 (V+)
- no-connect marks 1 -> 28
Other:
- note added: "components need to be added to increase hysteresis"
- note removed: "output components need to be done"
- title: (none) -> EDM Transistor Powersupply
