File: EDM_Powersupply.kicad_pcb (KiCad board)
At the start: 2 copper layers, 34 parts, among them IC1 ACSL-7210-06RE, J1 Screw_Terminal_01x02, J2 Screw_Terminal_01x02, J3 Screw_Terminal_01x02, J4 Screw_Terminal_01x02, J5 Conn_01x13_Pin, J6 Conn_01x07_Pin, U1 L7805, U2 STGAP2SM, U5 TLV3501AID, U6 MGJ2D241505SC, U7 MGJ2D241505SC

Commit message: good
Parts:
- added HS1: Heatsink, Heatsink:Heatsink_Fischer_SK104-STCB_35x13mm__2xDrill3.5mm_ScrewM3, F.Cu at (84.0, 80.0)
- added J7: Conn_01x03_Pin, Connector_PinHeader_2.54mm:PinHeader_1x03_P2.54mm_Vertical, F.Cu at (50.6, 154.4)
- added Q1: IPW65R037C6, IPW65R037C6:IPW65R037C6, F.Cu at (158.0, 96.0)
- added U4: RASPBERRY_PI_PICO, RASPBERRY_PI_PICO:RASPBERRY_PI_PICO, F.Cu at (77.1, 133.9)
- C1: renamed from C9; footprint Capacitor_SMD:C_0805_2012Metric_Pad1.18x1.45mm_HandSolder -> Capacitor_THT:CP_Radial_D10.0mm_P7.50mm
- C11: renamed from C5; footprint Capacitor_SMD:C_0805_2012Metric_Pad1.18x1.45mm_HandSolder -> Capacitor_THT:CP_Radial_D10.0mm_P7.50mm
- C12: renamed from C7; footprint Capacitor_SMD:C_0805_2012Metric_Pad1.18x1.45mm_HandSolder -> Capacitor_THT:CP_Radial_D10.0mm_P7.50mm
- C3: renamed from C10; footprint Capacitor_SMD:C_0805_2012Metric_Pad1.18x1.45mm_HandSolder -> Capacitor_THT:CP_Radial_D10.0mm_P7.50mm
- C5: renamed from C2; footprint Capacitor_SMD:C_0805_2012Metric_Pad1.18x1.45mm_HandSolder -> Capacitor_THT:CP_Radial_D10.0mm_P7.50mm
- C8: value 100n -> 0.1u
- IC1: footprint Connector_PinHeader_2.54mm:PinHeader_1x13_P2.54mm_Vertical -> ACSL-7210-06RE:ACSL-7210-06RE
- J2: renamed from J4; footprint TerminalBlock_4Ucon:TerminalBlock_4Ucon_1x02_P3.50mm_Vertical -> TerminalBlock:TerminalBlock_Altech_AK300-2_P5.00mm
- J3: footprint TerminalBlock_4Ucon:TerminalBlock_4Ucon_1x02_P3.50mm_Vertical -> TerminalBlock:TerminalBlock_Altech_AK300-2_P5.00mm
- J4: renamed from J1; footprint TerminalBlock_4Ucon:TerminalBlock_4Ucon_1x02_P3.50mm_Vertical -> TerminalBlock:TerminalBlock_Altech_AK300-2_P5.00mm
- J5: renamed from J2; footprint TerminalBlock_4Ucon:TerminalBlock_4Ucon_1x02_P3.50mm_Vertical -> TerminalBlock:TerminalBlock_Altech_AK300-2_P5.00mm
- moved J1 166.6 mm to (176.5, 146.9), turned to 180 degrees
- moved IC1 133.8 mm to (123.0, 123.5)
- moved J2 111.2 mm to (53.1, 80.9), turned to 90 degrees
- moved J6 104.4 mm to (48.1, 125.1)
- moved R9 99.5 mm to (136.5, 153.3), turned to 90 degrees
- moved U6 92.4 mm to (116.0, 147.9)
- moved C12 87.1 mm to (149.0, 146.2), turned to -90 degrees
- moved U5 84.2 mm to (144.8, 129.9), turned to 180 degrees
- moved C11 74.2 mm to (153.5, 136.5)
- moved R10 69.8 mm to (140.5, 145.8), turned to -90 degrees
- moved U1 69.5 mm to (116.3, 100.4)
- moved R7 69.3 mm to (159.9, 126.5), turned to 180 degrees
- moved R8 68.9 mm to (150.1, 136.5), turned to 180 degrees
- moved C9 65.2 mm to (117.0, 120.4)
- moved C8 60.9 mm to (132.5, 124.3), turned to 180 degrees
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- renumbered C13 to C10, C11 to C2, C1 to C4, C3 to C6, C12 to C7, C6 to C9, J5 to J1, R4 to R1, R9 to R10, R1 to R3, R5 to R4, R10 to R5, R3 to R9, U6 to U1, U1 to U2, U2 to U3, U7 to U6
Connections:
- net Net-(U2-GOFF) renamed /GOFF
- net Net-(U2-GON) renamed /GON
- net Net-(U2-IN+) renamed /IN+
- net Net-(U7-+VOUT) renamed /+VOUT
- C1 pad 2: Source -> 0V
- C3 pad 1: Source -> 0V
- C7 pad 1: Source -> 0V
- J1 pad 10: Source -> 0V
- J1 pad 6: Source -> unconnected-(J1-Pin_6-Pad6)
- J5 pad 2: Source -> 0V
- J6 pad 1: unconnected-(J6-Pin_1-Pad1) -> PWM
- J6 pad 2: unconnected-(J6-Pin_2-Pad2) -> DigitalMeasureLow
- J6 pad 3: unconnected-(J6-Pin_3-Pad3) -> MeasRefPWMLow
- J6 pad 4: unconnected-(J6-Pin_4-Pad4) -> +3.3V
- J6 pad 5: unconnected-(J6-Pin_5-Pad5) -> +5V
- J6 pad 6: unconnected-(J6-Pin_6-Pad6) -> +24V
- J6 pad 7: unconnected-(J6-Pin_7-Pad7) -> GNDS
- R5 pad 1: Source -> 0V
- U1 pad 6: Source -> 0V

Commit message: PCB Done?
Parts:
- added H1: MountingHole, MountingHole:MountingHole_3.2mm_M3, F.Cu at (71.5, 148.5)
- added H2: MountingHole, MountingHole:MountingHole_3.2mm_M3, F.Cu at (164.0, 155.0)
- added H3: MountingHole, MountingHole:MountingHole_3.2mm_M3, F.Cu at (151.5, 86.5)
- added H4: MountingHole, MountingHole:MountingHole_3.2mm_M3, F.Cu at (112.5, 89.5)
- moved J7 41.1 mm to (70.0, 118.2), turned to 180 degrees
- moved R1 31.5 mm to (111.0, 126.2), turned to 90 degrees
- moved J2 29.9 mm to (73.0, 103.2)
- moved J6 21.9 mm to (70.0, 125.0)
- moved R4 20.3 mm to (106.5, 126.2), turned to 90 degrees
- moved U4 13.9 mm to (90.9, 132.3)
- moved C4 13.4 mm to (93.5, 101.9)
- moved U2 13.4 mm to (92.5, 98.0)
- moved C5 12.0 mm to (102.9, 101.4)
- moved C8 8.68 mm to (138.0, 131.0)
- moved C7 8.23 mm to (161.5, 88.3)
- moved J3 8.23 mm to (169.5, 109.3)
- moved J4 8.23 mm to (169.5, 97.3)
- moved J5 8.23 mm to (169.5, 85.6)
- moved J1 8.23 mm to (174.0, 154.7)
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Connections:
- J5 pad 1: VoltageSense -> 0V
- J5 pad 2: 0V -> VoltageSense
Routing:
- net +24V: track 0.00 -> 135.3 mm, vias 0 -> 2
- net +3.3V: track 0.00 -> 124.2 mm, vias 0 -> 6
- net +5V: track 0.00 -> 109.9 mm, vias 0 -> 2
- net +15V: track 0.00 -> 92.1 mm, vias 0 -> 6
- net PWM: track 0.00 -> 91.6 mm, vias 0 -> 5
- net H+3.3V: track 0.00 -> 88.0 mm, vias 0 -> 6
- net -5V: track 0.00 -> 87.7 mm, vias 0 -> 4
- net VoltageSense: track 0.00 -> 83.6 mm, vias 0 -> 1
- net DigitalMeasureHigh: track 0.00 -> 83.3 mm
- net SDA: track 0.00 -> 81.6 mm
- net SCL: track 0.00 -> 78.3 mm
- net DigitalMeasureLow: track 0.00 -> 74.4 mm, vias 0 -> 2
- net MeasRefPWMLow: track 0.00 -> 74.2 mm, vias 0 -> 2
- net Gate: track 0.00 -> 73.0 mm
- net MeasRefPWMHigh: track 0.00 -> 67.8 mm, vias 0 -> 4
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- added copper zone on F.Cu, net +VDC
- added copper zone on B.Cu, net 0V
- added copper zone on B.Cu, net GND
- added copper zone on B.Cu, net GNDS
- added copper zone on F.Cu, net VoltageSense
Other:
- board outline added: 116.5 x 85 mm
- board text added: "+24"
- board text added: "-"
- board text added: "-5 0 15"
- board text added: "24V"
- board text added: "Current Limit"
- board text added: "GND"
- board text added: "OUTPUT+"
- board text added: "VDC+ IN"

Commit message: final?
Parts:
- removed C7: 0.1u, Capacitor_SMD:C_0805_2012Metric_Pad1.18x1.45mm_HandSolder
- removed HS1: Heatsink, Heatsink:Heatsink_Fischer_SK104-STCB_35x13mm__2xDrill3.5mm_ScrewM3
- added D1: D, Diode_THT:D_DO-15_P10.16mm_Horizontal, F.Cu at (164.1, 79.8)
- moved H4 36.2 mm to (76.6, 84.6)
- moved R5 25.2 mm to (131.8, 79.4), turned to 0 degrees
- moved Q1 13.6 mm to (147.8, 91.2), turned to 0 degrees
- moved H3 8.63 mm to (157.4, 80.2)
- moved C1 5.82 mm to (134.8, 93.6), turned to 0 degrees
- moved R2 3.63 mm to (131.8, 86.2)
- moved R3 3.42 mm to (131.8, 82.8)
Connections:
- J1 pad 6: unconnected-(J1-Pin_6-Pad6) -> +VOUT
- J5 pad 1: 0V -> VoltageSense
- J5 pad 2: VoltageSense -> 0V
- R9 pad 1: /+VOUT -> +VOUT
- U6 pad 7: /+VOUT -> +VOUT
Routing:
- net +VOUT: track 0.00 -> 54.9 mm, vias 0 -> 2
- net Gate: track 73.0 -> 83.9 mm
- net +15V: track 92.1 -> 82.5 mm
- net /+VOUT: track 8.80 -> 0.00 mm
- net 0V: track 52.7 -> 46.9 mm, vias 1 -> 0
- net /GON: track 10.9 -> 6.93 mm
- net /GOFF: track 10.2 -> 7.10 mm
Other:
- board text added: "+15V"
- board text added: "+24V"
- board text added: "+3.3V"
- board text added: "+5V"
- board text added: "+VDC"
- board text added: "-5V"
- board text added: "0V"
- board text added: "COMP+"
- board text added: "COMP-"
- board text added: "DigMLow"
- board text added: "DigitalMeasureHigh"
- board text added: "GNDS"
- board text added: "Gate"
- board text added: "Gate Driver"
- board text added: "H+3.3V"
- board text added: "HIGH"
- board text added: "ISOLATED"
- board text added: "LOW"
- board text added: "MRefLow"
- board text added: "MeasRefPWMHigh"
- board text added: "OPTOCOUPLER"
- board text added: "PWM"
- board text added: "SCL"
- board text added: "SDA"
- board text added: "VOUT+"
- board text added: "VoltageSense"

Commit message: stash
Parts:
- moved C11 71.2 mm to (111.3, 79.1)
- moved C6 71.2 mm to (74.6, 23.8)
- moved C8 71.2 mm to (95.8, 73.6)
- moved H1 71.2 mm to (29.3, 91.1)
- moved H2 71.2 mm to (121.8, 97.6)
- moved H3 71.2 mm to (115.2, 22.8)
- moved IC1 71.2 mm to (80.8, 66.1)
- moved J2 71.2 mm to (30.8, 45.8)
- moved J3 71.2 mm to (127.3, 51.9)
- moved J4 71.2 mm to (127.3, 39.9)
- moved J5 71.2 mm to (127.3, 28.2)
- moved J7 71.2 mm to (27.8, 60.8)
- moved Q1 71.2 mm to (105.6, 33.8)
- moved R1 71.2 mm to (68.8, 68.8)
- moved R10 71.2 mm to (98.3, 88.4)
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