File: Laars.kicad_sch (KiCad schematic)
At the start: 12 parts, among them Q1 NMOS, Q2 NPN

Commit message: working simulation
Connections:
- net GND renamed 0
Changed lines of the file:
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@@
+	(wire
+		(pts
+			(xy 162.56 123.19) (xy 162.56 121.92)
+		)
+		(stroke
+			(width 0)
+			(type default)
+		)
+	)
 	(wire
 		(pts
@@
 	(wire
 		(pts
-			(xy 123.19 120.65) (xy 134.62 120.65)
+			(xy 162.56 121.92) (xy 167.64 121.92)
 		)
 		(stroke
@@
 	(wire
 		(pts
-			(xy 134.62 100.33) (xy 134.62 102.87)
+			(xy 123.19 120.65) (xy 134.62 120.65)
 		)
 		(stroke
@@
 	(wire
 		(pts
-			(xy 105.41 107.95) (xy 121.92 107.95)
+			(xy 134.62 100.33) (xy 134.62 102.87)
 		)
 		(stroke
@@
 	(wire
 		(pts
-			(xy 110.49 115.57) (xy 121.92 115.57)
+			(xy 105.41 107.95) (xy 121.92 107.95)
 		)
 		(stroke
@@
 	(wire
 		(pts
-			(xy 133.35 115.57) (xy 133.35 113.03)
+			(xy 110.49 115.57) (xy 121.92 115.57)
 		)
 		(stroke
@@
 		)
 	)
+	(wire
+		(pts
+			(xy 133.35 115.57) (xy 133.35 113.03)
+		)
+		(stroke
+			(width 0)
+			(type default)
+		)
+	)
 	(label "uit"
 		(at 134.62 113.03 0)
@@
 	)
 	(symbol
+		(lib_id "Simulation_SPICE:0")
+		(at 162.56 123.19 0)
+		(unit 1)
+		(exclude_from_sim no)
+		(in_bom yes)
+		(on_board yes)
+		(dnp no)
+		(fields_autoplaced yes)
+		(property "Reference" "#GND01"
+			(at 162.56 128.27 0)
+			(effects
+				(font
+					(size 1.27 1.27)
+				)
+				(hide yes)
+			)
+		)
+		(property "Value" "0"
+			(at 162.56 120.65 0)
+			(effects
+				(font
+					(size 1.27 1.27)
+				)
+			)
+		)
+		(property "Footprint" ""
+			(at 162.56 123.19 0)
+			(effects
+				(font
+					(size 1.27 1.27)
+				)
+				(hide yes)
+			)
+		)
+		(property "Datasheet" "https://ngspice.sourceforge.io/docs/ngspice-html-manual/manual.xhtml#subsec_Circuit_elements__device"
+			(at 162.56 133.35 0)
+			(effects
+				(font
+					(size 1.27 1.27)
+				)
+				(hide yes)
+			)
+		)
+		(property "Description" "0V reference potential for simulation"
+			(at 162.56 130.81 0)
+			(effects
+				(font
+					(size 1.27 1.27)
+				)
+				(hide yes)
+			)
+		)
+		(pin "1"
+		)
+		(instances
+			(project "Laars"
+				(path "/4688d223-df16-4fb7-9dfd-c1858c1588a6"
+					(reference "#GND01")
+					(unit 1)
+				)
+			)
+		)
+	)
+	(symbol
 		(lib_id "Simulation_SPICE:VPULSE")
 		(at 90.17 134.62 0)
@@
 					(unit 1)
 				)
+			)
+		)
+	)
+	(symbol
+		(lib_id "power:GND")
+		(at 167.64 121.92 0)
+		(unit 1)
+		(exclude_from_sim no)
+		(in_bom yes)
+		(on_board yes)
+		(dnp no)
+		(fields_autoplaced yes)
+		(property "Reference" "#PWR05"
+			(at 167.64 128.27 0)
+			(effects
+				(font
+					(size 1.27 1.27)
+				)
+				(hide yes)
+			)
+		)
+		(property "Value" "GND"
+			(at 167.64 127 0)
+			(effects
+				(font
+					(size 1.27 1.27)
+				)
+			)
+		)
+		(property "Footprint" ""
+			(at 167.64 121.92 0)
+			(effects
+				(font
+					(size 1.27 1.27)
+				)
+				(hide yes)
+			)
+		)
+		(property "Datasheet" ""
+			(at 167.64 121.92 0)
+			(effects
+				(font
+					(size 1.27 1.27)
+				)
+				(hide yes)
+			)
+		)
+		(property "Description" "Power symbol creates a global label with name \"GND\" , ground"
+			(at 167.64 121.92 0)
+			(effects
+				(font
+					(size 1.27 1.27)
+				)
+				(hide yes)
+			)
+		)
+		(pin "1"
+		)
+		(instances
+			(project "Laars"
+				(path "/4688d223-df16-4fb7-9dfd-c1858c1588a6"
+					(reference "#PWR05")
+					(unit 1)
+				)

Commit message: V4
Parts:
- removed D1, D2: D, symbol Device:D
- removed Q2: NPN, symbol Simulation_SPICE:NPN
- removed R4: 220, symbol Device:R
- removed V1: 24, symbol Simulation_SPICE:VDC
- removed V3: VPULSE, symbol Simulation_SPICE:VPULSE
- added L1: 3u, symbol Device:L
- added V4: VPULSE, symbol Simulation_SPICE:VPULSE
- C1: value 100n -> 47n
- R2: value 1k -> 10k
- R3: value 2.2k -> 1.2
Connections:
- net at V2.1: now also C1.1, R1.1; no longer Q1.1 (D)
- net at R3.2: now also V4.1
- net at R3.1: now also Q1.2 (G), R2.1
- net 0: no longer names the net of R1.2
- net 0: now also L1.1; no longer V2.2
- removed net 1: C1.1, R2.1
- net gate renamed GND
- net GND: now also Q1.3 (S), V2.2, V4.2; no longer Q1.2 (G)
- removed net uit: C1.2, Q1.3 (S), R1.1
- new net: C1.2, L1.2, Q1.1 (D)
Other:
- moved on the sheet: V2
